Commit message: fully ingrated wrist into urdf, works with angles commands

File: install/main_arm_package/share/main_arm_package/urdf/arm.urdf (robot description, URDF)
Before this commit: robot arm_robot, 6 links, 5 joints
Links:
- removed link main_arm
- removed link tip_arm
- added link elbow_arm; collision cylinder length=0.35 radius=0.03; visual cylinder length=0.35 radius=0.03
- added link wrist_arm; collision cylinder length=0.10 radius=0.010; visual cylinder length=0.15 radius=0.015
- added link wrist_link; collision sphere radius=0.035; visual sphere radius=0.035
- link shoulder_arm: geometry collision cylinder length=0.4 radius=0.03; visual cylinder length=0.4 radius=0.03
Joints:
- removed joint body_arm_joint
- removed joint elbow_shoulder_joint
- removed joint tip_arm_joint
- added joint elbow_arm_joint: type continuous, parent elbow_link, child elbow_arm, origin xyz=0 0 0.035 rpy=0 0 0, axis 0 0 1
- added joint elbow_main_joint: type revolute, parent shoulder_arm, child elbow_link, origin xyz=0 0 0.35 rpy=0 0 0, axis 0 1 0, limit lower=-1.57 upper=1.57 effort=10 velocity=1
- added joint wrist_arm_joint: type continuous, parent wrist_link, child wrist_arm, origin xyz=0 0 0.005 rpy=0 0 0, axis 0 0 1
- added joint wrist_main_joint: type revolute, parent elbow_arm, child wrist_link, origin xyz=0 0 0.32 rpy=0 0 0, axis 0 1 0, limit lower=-1.57 upper=1.57 effort=10 velocity=1
- joint shoulder_arm_joint: origin xyz=0 0 0 rpy=0 0 0 -> xyz=0 0 0.04 rpy=0 0 0
- joint shoulder_main_joint: origin xyz=0 0 0.3 rpy=0 0 0 -> xyz=0 0 0.06 rpy=0 0 0; parent main_arm -> robot_base

Commit message: added the spin angles, the arm could access the z axis now

File: install/main_arm_package/share/main_arm_package/urdf/arm.urdf (robot description, URDF)
Before this commit: robot arm_robot, 7 links, 6 joints
Links:
- added link spin_arm; collision cylinder length=0.1 radius=0.03; visual cylinder length=0.1 radius=0.03
- added link spin_link; collision sphere radius=0.035; visual sphere radius=0.035
Joints:
- added joint spin_arm_joint: type continuous, parent spin_link, child spin_arm, origin xyz=0 0 0.02 rpy=0 0 0, axis 0 0 1
- added joint spin_main_joint: type revolute, parent robot_base, child spin_link, origin xyz=0 0 0.06 rpy=0 0 0, axis 0 0 1, limit lower=-1.57 upper=1.57 effort=10 velocity=1
- joint shoulder_main_joint: origin xyz=0 0 0.06 rpy=0 0 0 -> xyz=0 0 0.1 rpy=0 0 0; parent robot_base -> spin_arm

Commit message: working x y requests instead of angles, need z for height

File: install/main_arm_package/share/main_arm_package/urdf/arm.urdf (robot description, URDF)
Before this commit: robot arm_robot, 9 links, 8 joints
Joints:
- joint spin_main_joint: limit lower=-1.57 upper=1.57 effort=10 velocity=1 -> lower=-3.14159 upper=3.14159 effort=10 velocity=1

Commit message: added grip capability (close/open)

File: install/main_arm_package/share/main_arm_package/urdf/arm.urdf (robot description, URDF)
Before this commit: robot arm_robot, 9 links, 8 joints
Links:
- added link gripper_base; collision box size=0.02 0.02 0.02; visual box size=0.02 0.08 0.02
- added link gripper_left_finger; collision box size=0.015 0.015 0.045; visual box size=0.015 0.015 0.045
- added link gripper_right_finger; collision box size=0.015 0.015 0.045; visual box size=0.015 0.015 0.045
- link wrist_arm: geometry collision cylinder length=0.05 radius=0.012; visual cylinder length=0.05 radius=0.012
Joints:
- added joint gripper_base_joint: type fixed, parent wrist_arm, child gripper_base, origin xyz=0 0 0.01 rpy=0 0 0
- added joint gripper_left_finger_joint: type prismatic, parent gripper_base, child gripper_left_finger, origin xyz=0 0 0.045 rpy=0 0 0, axis 0 1 0, limit lower=0.0 upper=0.04 effort=5 velocity=0.1
- added joint gripper_right_finger_joint: type prismatic, parent gripper_base, child gripper_right_finger, origin xyz=0 0 0.045 rpy=0 0 0, axis 0 1 0, limit lower=0.0 upper=0.04 effort=5 velocity=0.1
- joint wrist_arm_joint: origin xyz=0 0 0.005 rpy=0 0 0 -> xyz=0 0 0.025 rpy=0 0 0

Commit message: gazebo launch file and movement in the gazebo terminal working

File: install/main_arm_package/share/main_arm_package/urdf/arm.urdf (robot description, URDF)
Before this commit: robot arm_robot, 12 links, 11 joints
Links:
- added link world
- link elbow_arm: mass None -> 0.12
- link elbow_link: mass None -> 0.05
- link gripper_base: mass None -> 0.03
- link gripper_left_finger: mass None -> 0.01
- link gripper_right_finger: mass None -> 0.01
- link robot_base: mass None -> 0.5
- link shoulder_arm: mass None -> 0.15
- link shoulder_link: mass None -> 0.05
- link spin_arm: mass None -> 0.05
- link spin_link: mass None -> 0.05
- link wrist_arm: mass None -> 0.02
- link wrist_link: mass None -> 0.03
Joints:
- added joint world_joint: type fixed, parent world, child robot_base, origin xyz=0 0 0.05 rpy=0 0 0
- joint elbow_arm_joint: axis 0 0 1 -> (none); type continuous -> fixed
- joint gripper_left_finger_joint: limit lower=0.0 upper=0.04 effort=5 velocity=0.1 -> lower=-0.04 upper=0.04 effort=5 velocity=0.1
- joint gripper_right_finger_joint: axis 0 1 0 -> 0 -1 0; limit lower=0.0 upper=0.04 effort=5 velocity=0.1 -> lower=-0.04 upper=0.04 effort=5 velocity=0.1
- joint shoulder_arm_joint: axis 0 0 1 -> (none); type continuous -> fixed
- joint spin_arm_joint: axis 0 0 1 -> (none); type continuous -> fixed
- joint wrist_arm_joint: axis 0 0 1 -> (none); type continuous -> fixed

Commit message: added contact sensors on grippers

File: install/main_arm_package/share/main_arm_package/urdf/arm.urdf (robot description, URDF)
Before this commit: robot arm_robot, 13 links, 12 joints
Joints:
- joint elbow_main_joint: limit lower=-1.57 upper=1.57 effort=10 velocity=1 -> lower=-2.356 upper=2.356 effort=10 velocity=1
- joint wrist_main_joint: limit lower=-1.57 upper=1.57 effort=10 velocity=1 -> lower=-2.094 upper=2.094 effort=10 velocity=1

File: src/main_arm_package/urdf/arm.urdf (robot description, URDF)
Before this commit: robot arm_robot, 13 links, 12 joints
Joints:
- joint elbow_main_joint: limit lower=-1.57 upper=1.57 effort=10 velocity=1 -> lower=-2.356 upper=2.356 effort=10 velocity=1
- joint wrist_main_joint: limit lower=-1.57 upper=1.57 effort=10 velocity=1 -> lower=-2.094 upper=2.094 effort=10 velocity=1
